File: DevelopmentBoards/ADS_v5/Sanket Deployment board/sanket.kicad_sch (KiCad schematic)
At the start: 43 parts, among them J1 Conn_01x06_Socket, J2 DeploymentInhibit, J3 Conn_01x06_Socket, J4 CurrentSense, J5 Deployer2, J6 Conn_01x01_Socket, Q1 ZXMP6A17GQTA, U1 SN74LVC1G17QDCKRQ1, U2 TPS54260DGQ, U3 TPS25200QDRVTQ1

Commit message: add bom
Parts:
- C5: value 22µF -> 22uF
Changed lines of the file:
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@@
 			)
 		)
-		(property "Value" "22µF"
+		(property "Value" "22uF"
 			(at 183.388 111.506 0)
 			(effects
